Commit message: franka panda simulation model updates

File: franka/description/manipulator.control.xacro (robot description, xacro)
@@ -15,5 +15,7 @@
                 <!-- <param name="max">2.8973</param> -->
             </command_interface>
-            <state_interface name="position" />
+            <state_interface name="position">
+            	<param name="initial_value">-1.57</param>
+            </state_interface>
             <state_interface name="velocity" />
             <state_interface name="effort" />
@@ -24,5 +26,7 @@
                 <!-- <param name="max">1.7628</param> -->
             </command_interface>
-            <state_interface name="position" />
+            <state_interface name="position">
+            	<param name="initial_value">0.67</param>
+            </state_interface>
             <state_interface name="velocity" />
             <state_interface name="effort" />
@@ -33,5 +37,7 @@
                 <!-- <param name="max">2.8973</param> -->
             </command_interface>
-            <state_interface name="position" />
+            <state_interface name="position">
+            	<param name="initial_value">0.0</param>
+            </state_interface>
             <state_interface name="velocity" />
             <state_interface name="effort" />
@@ -42,5 +48,7 @@
                 <!-- <param name="max">-0.0698</param> -->
             </command_interface>
-            <state_interface name="position" />
+            <state_interface name="position">
+            	<param name="initial_value">0.0</param>
+            </state_interface>
             <state_interface name="velocity" />
             <state_interface name="effort" />
@@ -51,5 +59,7 @@
                 <!-- <param name="max">2.8973</param> -->
             </command_interface>
-            <state_interface name="position" />
+            <state_interface name="position">
+            	<param name="initial_value">0.0</param>
+            </state_interface>
             <state_interface name="velocity" />
             <state_interface name="effort" />
@@ -60,5 +70,7 @@
                 <!-- <param name="max">3.7525</param> -->
             </command_interface>
-            <state_interface name="position" />
+            <state_interface name="position">
+            	<param name="initial_value">1.3</param>
+            </state_interface>
             <state_interface name="velocity" />
             <state_interface name="effort" />
@@ -69,5 +81,29 @@
                 <!-- <param name="max">3.7525</param> -->
             </command_interface>
-            <state_interface name="position" />
+            <state_interface name="position">
+            	<param name="initial_value">-2.3</param>
+            </state_interface>
+            <state_interface name="velocity" />
+            <state_interface name="effort" />
+        </joint>
+        <joint name="panda_finger_joint1">
+            <command_interface name="position">
+                <!-- <param name="min">-0.0175</param> -->
+                <!-- <param name="max">3.7525</param> -->
+            </command_interface>
+            <state_interface name="position">
+            	<param name="initial_value">0.0</param>
+            </state_interface>
+            <state_interface name="velocity" />
+            <state_interface name="effort" />
+        </joint>
+        <joint name="panda_finger_joint2">
+            <command_interface name="position">
+                <!-- <param name="min">-0.0175</param> -->
+                <!-- <param name="max">3.7525</param> -->
+            </command_interface>
+            <state_interface name="position">
+            	<param name="initial_value">0.0</param>
+            </state_interface>
             <state_interface name="velocity" />
             <state_interface name="effort" />

File: franka/description/manipulator.gazebo.xacro (robot description, xacro)
@@ -13,4 +13,6 @@
             <joint_name>panda_joint6</joint_name>
             <joint_name>panda_joint7</joint_name>
+            <joint_name>panda_finger_joint1</joint_name>
+            <joint_name>panda_finger_joint2</joint_name>
         </plugin>
     </gazebo>

File: franka/description/manipulator.urdf.xacro (robot description, xacro)
@@ -8,11 +8,11 @@
     <!-- Include arm and hand xacro files-->
     <xacro:include filename="$(find franka)/description/panda_arm.xacro" />
-    <xacro:include filename="$(find franka)/description/panda_hand.xacro" />
+    <xacro:include filename="$(find franka)/description/panda_hand_gripper.xacro" />
     <xacro:include filename="$(find franka)/description/rgbd_camera.xacro" />
     <!-- call the arm macro-->
     <xacro:panda_arm xyz="0 0 0" rpy="0 0 0" connected_base="${connected_base}"/>
     <!-- call the hand macro-->
-    <xacro:panda_hand ns="panda" rpy="0 0 ${-pi/4}" connected_to="panda_link8" />
-    <xacro:rgbd_camera rpy="0 ${-pi/2} 0" connected_to="panda_finger" />
+    <xacro:panda_hand_gripper ns="panda" rpy="0 0 ${-pi/4}" connected_to="panda_link8" />
+    <xacro:rgbd_camera rpy="0 ${-pi/2} 0" connected_to="panda_hand" />
   </xacro:macro>
 </robot>

File: franka/description/mobile_manipulator.control.xacro (robot description, xacro)
@@ -10,5 +10,7 @@
                 <!-- <param name="max">2.8973</param> -->
             </command_interface>
-            <state_interface name="position" />
+            <state_interface name="position">
+            	<param name="initial_value">-1.57</param>
+            </state_interface>
             <state_interface name="velocity" />
             <state_interface name="effort" />
@@ -19,5 +21,7 @@
                 <!-- <param name="max">1.7628</param> -->
             </command_interface>
-            <state_interface name="position" />
+            <state_interface name="position">
+            	<param name="initial_value">0.67</param>
+            </state_interface>
             <state_interface name="velocity" />
             <state_interface name="effort" />
@@ -28,5 +32,7 @@
                 <!-- <param name="max">2.8973</param> -->
             </command_interface>
-            <state_interface name="position" />
+            <state_interface name="position">
+            	<param name="initial_value">0.0</param>
+            </state_interface>
             <state_interface name="velocity" />
             <state_interface name="effort" />
@@ -37,5 +43,7 @@
                 <!-- <param name="max">-0.0698</param> -->
             </command_interface>
-            <state_interface name="position" />
+            <state_interface name="position">
+            	<param name="initial_value">0.0</param>
+            </state_interface>
             <state_interface name="velocity" />
             <state_interface name="effort" />
@@ -46,5 +54,7 @@
                 <!-- <param name="max">2.8973</param> -->
             </command_interface>
-            <state_interface name="position" />
+            <state_interface name="position">
+            	<param name="initial_value">0.0</param>
+            </state_interface>
             <state_interface name="velocity" />
             <state_interface name="effort" />
@@ -55,5 +65,7 @@
                 <!-- <param name="max">3.7525</param> -->
             </command_interface>
-            <state_interface name="position" />
+            <state_interface name="position">
+            	<param name="initial_value">1.3</param>
+            </state_interface>
             <state_interface name="velocity" />
             <state_interface name="effort" />
@@ -64,5 +76,29 @@
                 <!-- <param name="max">3.7525</param> -->
             </command_interface>
-            <state_interface name="position" />
+            <state_interface name="position">
+            	<param name="initial_value">-2.3</param>
+            </state_interface>
+            <state_interface name="velocity" />
+            <state_interface name="effort" />
+        </joint>
+        <joint name="panda_finger_joint1">
+            <command_interface name="position">
+                <!-- <param name="min">-0.0175</param> -->
+                <!-- <param name="max">3.7525</param> -->
+            </command_interface>
+            <state_interface name="position">
+            	<param name="initial_value">0.0</param>
+            </state_interface>
+            <state_interface name="velocity" />
+            <state_interface name="effort" />
+        </joint>
+        <joint name="panda_finger_joint2">
+            <command_interface name="position">
+                <!-- <param name="min">-0.0175</param> -->
+                <!-- <param name="max">3.7525</param> -->
+            </command_interface>
+            <state_interface name="position">
+            	<param name="initial_value">0.0</param>
+            </state_interface>
             <state_interface name="velocity" />
             <state_interface name="effort" />

File: franka/description/rgbd_camera.xacro (robot description, xacro)
@@ -1,5 +1,5 @@
 <?xml version="1.0" encoding="utf-8"?>
 <robot xmlns:xacro="http://www.ros.org/wiki/xacro" name="rgbd_camera">
-    <xacro:macro name="rgbd_camera" params="connected_to:='' rpy:='0 -1.57 0' xyz:='0 0 0' ">
+    <xacro:macro name="rgbd_camera" params="connected_to:='' rpy:='0 -1.57 0' xyz:='0 0 0.112' ">
         <xacro:unless value="${connected_to == ''}">
             <joint name="tip_camera_joint" type="fixed">
